Commit message: Changes to be committed: 	new file:   p12/robutler_bringup/CMakeLists.txt 	new file:   p12/robutler_bringup/config/rviz.rviz 	new file:   p12/robutler_bringup/launch/gazebo.launch 	new file:   p12/robutler_bringup/launch/spawn.launch 	new file:   p12/robutler_bringup/package.xml 	renamed:    p12/robutler_description/urdf/turtlebot3_waffle_pi.gazebo.xacro -> p12/robutler_description/urdf/robutler.gazebo.xacro 	renamed:    p12/robutler_description/urdf/turtlebot3_waffle_pi.urdf.xacro -> p12/robutler_description/urdf/robutler.urdf.xacro

File: p12/robutler_description/urdf/robutler.gazebo.xacro (robot description, xacro)
@@ -5,5 +5,5 @@
   <xacro:arg name="imu_visual"    default="false"/>
   <gazebo reference="base_link">
-    <material>Gazebo/DarkGrey</material>
+    <material>Gazebo/Red</material>
   </gazebo>
   <gazebo reference="wheel_left_link">
@@ -103,9 +103,9 @@
   </gazebo>
   <gazebo reference="base_scan">
-    <material>Gazebo/FlatBlack</material>
+    <material>Gazebo/Blue</material>
     <sensor type="ray" name="lds_lfcd_sensor">
       <pose>0 0 0 0 0 0</pose>
       <visualize>$(arg laser_visual)</visualize>
-      <update_rate>5</update_rate>
+      <update_rate>5</update_rate>s
       <ray>
         <scan>

File: p12/robutler_description/urdf/robutler.urdf.xacro (robot description, xacro)
@@ -1,6 +1,6 @@
 <?xml version="1.0" ?>
 <robot name="turtlebot3_waffle_pi" xmlns:xacro="http://ros.org/wiki/xacro">
-  <xacro:include filename="$(find turtlebot3_description)/urdf/common_properties.xacro"/>
-  <xacro:include filename="$(find turtlebot3_description)/urdf/turtlebot3_waffle_pi.gazebo.xacro"/>
+  <xacro:include filename="$(find robutler_description)/urdf/common_properties.xacro"/>
+  <xacro:include filename="$(find robutler_description)/urdf/robutler.gazebo.xacro"/>
   <link name="base_footprint"/>
   <joint name="base_joint" type="fixed">
